Commit message: odom frame finally works

File: seesaw_ros2/urdf/seesaw.urdf (robot description, URDF)
Before this commit: robot seesaw, 3 links, 2 joints
Links:
- removed link imu_link
Joints:
- removed joint base_to_imu

Commit message: back to stability with cyclonedds

File: seesaw_ros2/urdf/seesaw.urdf (robot description, URDF)
Before this commit: robot seesaw, 2 links, 1 joints
Links:
- added link imu_link; visual box size=0.03 0.02 0.01
Joints:
- added joint base_to_imu: type fixed, parent base_link, child imu_link, origin xyz=0 0 0.02 rpy=0 0 0
- joint base_to_lidar: origin xyz=0.015 0 0.04 -> xyz=0.015 0 0.04 rpy=0 0 0

Commit message: Still kinda bad

File: seesaw_ros2/urdf/seesaw.urdf (robot description, URDF)
Before this commit: robot seesaw, 3 links, 2 joints
Links:
- added link pitch_pivot_link
- link base_link: geometry 
- link imu_link: geometry visual box size=0.040 0.020 0.003
- link lidar_link: geometry visual cylinder length=0.070 radius=0.038
Joints:
- removed joint base_to_imu
- removed joint base_to_lidar
- added joint base_to_pitch_pivot: type fixed, parent base_link, child pitch_pivot_link, origin xyz=0 0 0 rpy=0 0 0
- added joint lidar_to_imu: type fixed, parent lidar_link, child imu_link, origin xyz=-0.054356 0 -0.021590 rpy=3.141592653589793 0 0
- added joint pitch_joint: type revolute, parent pitch_pivot_link, child lidar_link, origin xyz=0 0 0 rpy=0 0 0, axis 0 1 0, limit lower=-1.57 upper=1.57 effort=1.0 velocity=5.0
